File: Hardware/Trochi.kicad_pcb (KiCad board)
At the start: 2 copper layers, 19 x 26.2 mm, 53 parts, among them IC1 ICM-42688-P, J1 JST-SH, J2 JST-SH, J3 JST PH, J4 Conn_01x09, J5 Conn_01x09, J6 JST-SH, J7 JST-SH, Q1 AO3400A, Q2 AO3400A, Q3 AO3400A, Q4 AO3400A, Q5 AO3400A, U1 ME6211C33M5, U3 YX-SMD5020

Commit message: style: add logo and silkscreen artwork to PCB
Parts:
- added G***: LOGO, LOGO, F.Cu at (149.5, 96.7)
- added G***: LOGO, LOGO, F.Cu at (149.4, 106.7)
- added G***: LOGO, LOGO, F.Cu at (145.4, 106.0)
- added G***: LOGO, LOGO, B.Cu at (143.6, 110.1)
- added G***: LOGO, LOGO, B.Cu at (154.2, 110.3)
- added G***: LOGO, LOGO, B.Cu at (150.3, 107.1)
Other:
- board text added: "+"
- board text added: "-"

Commit message: feat: update fotogrpahy on pcb
Parts:
- moved G*** 0.45 mm to (145.3, 106.5), turned to 0 degrees
- moved G*** 0.37 mm to (149.2, 96.9), turned to 0 degrees
- moved G*** 0.36 mm to (150.4, 107.4)
- moved G*** 0.21 mm to (143.5, 110.0)
- moved G*** 0.16 mm to (149.5, 106.9), turned to 0 degrees
- moved G*** 0.05 mm to (154.2, 110.3)
